File: hardware/led_driver.kicad_pcb (KiCad board)
At the start: 4 copper layers, 24 x 41 mm, 43 parts, among them J1 CONN_01X01, J2 CONN_01X05, J3 CONN_01X05, J4 CONN_01X08, J5 CONN_01X08, J6 CONN_01X08, J7 CONN_01X08, J8 AVR-PDI-6A, P1 USB_A, U1 AP3211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

Commit message: Sorted out library references
Parts:
- added U8: ASEK-32.768kHz, Kuro:Crystal-3.2x2.5-ASEK-Series-Abracon, B.Cu at (152.9, 50.8)
- J2: footprint Primayer:B5B-ZR-SM4-TF -> Kuro:B5B-ZR-SM4-TF
- J3: value CONN_01X05 -> CONN_01X08; footprint Primayer:B5B-ZR-SM4-TF -> Kuro:B8B-ZR-SM4-TF
- J4, J5, J6, J7: footprint Primayer:B8B-ZR-SM4-TF -> Kuro:B8B-ZR-SM4-TF
- J8: footprint Primayer:3x2_1.27mm_SMD_header -> Kuro:3x2_1.27mm_SMD_header
- P1: footprint Primayer:Molex_47346-0001_Micro_USB_SMT -> Kuro:Molex_47346-0001_Micro_USB_SMT
- U7: footprint Primayer:KT3225T -> Kuro:KT3225T
- moved J1 2.02 mm to (150.6, 47.2)
- moved J3 1.99 mm to (159.5, 45.1)
Connections:
- J2 pad 3: /SCL -> /SCK
- J3 pad 3: /EXP_RX_SDA -> /SDA
- J3 pad 4: /EXP_TX_SCL -> /SCL
- J3 pad 5: GND -> /TX
- R4 pad 2: /EXP_RX_SDA -> /SDA
- R5 pad 2: /EXP_TX_SCL -> /SCL
- U2 pad 4: /EXP_TX_SCL -> /SCL
- U2 pad 5: /EXP_RX_SDA -> /SDA
- U4 pad 11: /SCL -> /SCK
- U4 pad 13: /EXP_TX_SCL -> /TX
- U4 pad 14: /EXP_RX_SDA -> /RX
- U4 pad 15: /EXP_TX_SCL -> /SCL
- U4 pad 16: /EXP_RX_SDA -> /SDA
- U5 pad 14: /SCL -> /SCK
- U6 pad 14: /SCL -> /SCK
Routing:
- net /SCK: track 0.00 -> 40.4 mm, vias 0 -> 3
- net /EXP_RX_SDA: track 37.2 -> 0.00 mm, vias 2 -> 0
- net /EXP_TX_SCL: track 34.2 -> 0.00 mm, vias 4 -> 0
- net /SDA: track 0.00 -> 32.8 mm, vias 0 -> 2
- net +3V3: track 44.7 -> 49.1 mm
- net /SCL: track 40.4 -> 36.2 mm, vias 3 -> 4
- net Net-(U4-Pad19): track 14.5 -> 18.8 mm
- net /TX: track 0.00 -> 3.91 mm, vias 0 -> 1
- net /R_CLK: track 33.9 -> 30.1 mm
- net /RX: track 0.00 -> 3.62 mm, vias 0 -> 1
- net /PDI_C: track 12.2 -> 13.7 mm
- net /SDO2: track 29.6 -> 28.1 mm
- net /PDI_D: track 15.2 -> 16.2 mm
- net Net-(C5-Pad1): track 9.30 -> 10.1 mm
- net +5V: track 50.4 -> 49.7 mm
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
Commit message: Preparing for production
Other:
- board text added: "Rev 1.0"
- board text added: "©2016 Paul Qureshi"
Changed lines of the file:
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@@
     (area 143.924999 18.924999 168.075001 60.075001)
     (thickness 1.6)
-    (drawings 217)
+    (drawings 225)
     (tracks 679)
     (zones 0)
@@
   (page A4)
   (title_block
-    (title "LED Driver Board")
+    (title "LED Driver Board with FM radio")
+    (date 2016-11-12)
     (rev 1.0)
+    (company Keio)
   )
   (layers
@@
     (1 PWR.Cu signal hide)
     (2 GND.Cu signal hide)
-    (31 B.Cu signal)
+    (31 B.Cu signal hide)
     (32 B.Adhes user)
     (33 F.Adhes user)
@@
     (41 Cmts.User user)
     (42 Eco1.User user)
-    (43 Eco2.User user)
+    (43 Eco2.User user hide)
     (44 Edge.Cuts user)
     (45 Margin user)
@@
     (pad_to_mask_clearance 0.2)
     (aux_axis_origin 0 0)
-    (visible_elements 7FFEFF9F)
+    (visible_elements 7FFEFB9F)
     (pcbplotparams
-      (layerselection 0x00030_80000001)
-      (usegerberextensions false)
+      (layerselection 0x01cc0_80000007)
+      (usegerberextensions true)
       (excludeedgelayer true)
       (linewidth 0.100000)
@@
       (plotinvisibletext false)
       (padsonsilk false)
-      (subtractmaskfromsilk false)
+      (subtractmaskfromsilk true)
       (outputformat 1)
       (mirror false)
       (drillshape 0)
       (scaleselection 1)
-      (outputdirectory ""))
+      (outputdirectory plot/))
   )
   (net 0 "")
@@
       (net 7 +3V3))
   )
+  (gr_text "Rev 1.0" (at 145.1 27.8 90) (layer Eco2.User)
+    (effects (font (size 1 1) (thickness 0.2)) (justify mirror))
+  )
+  (gr_circle (center 150.3 49.7) (end 150.7 49.7) (layer Eco2.User) (width 0.15))
+  (gr_line (start 150.9 52.3) (end 150.9 49.3) (layer Eco2.User) (width 0.15))
+  (gr_line (start 154.9 52.3) (end 150.9 52.3) (layer Eco2.User) (width 0.15))
+  (gr_line (start 154.9 49.3) (end 154.9 52.3) (layer Eco2.User) (width 0.15))
+  (gr_line (start 150.9 49.3) (end 154.9 49.3) (layer Eco2.User) (width 0.15))
+  (gr_text "©2016 Paul Qureshi" (at 167 25.7 90) (layer Eco2.User)
+    (effects (font (size 0.8 0.8) (thickness 0.1)) (justify mirror))
+  )
+  (gr_text "©2016 Paul Qureshi" (at 167 25.7 90) (layer B.Cu)
+    (effects (font (size 0.8 0.8) (thickness 0.1)) (justify mirror))
+  )
   (gr_line (start 152.3 46.8) (end 152.3 46) (layer Eco1.User) (width 0.15))
   (gr_line (start 152.3 46.8) (end 153.8 46.8) (layer Eco1.User) (width 0.15))
@@
   (gr_line (start 154.2 57.3) (end 155 57.3) (layer Eco2.User) (width 0.15))
   (gr_line (start 155 56.1) (end 154.2 56.1) (layer Eco2.User) (width 0.15))
-  (gr_circle (center 151.6 52) (end 152 52) (layer Eco2.User) (width 0.15))
+  (gr_circle (center 151.4 52.9) (end 151.8 52.9) (layer Eco2.User) (width 0.15))
   (gr_line (start 152 55.6) (end 152 52.4) (layer Eco2.User) (width 0.15))
   (gr_line (start 156 55.6) (end 152 55.6) (layer Eco2.User) (width 0.15))
@@
     (effects (font (size 1.3 1.3) (thickness 0.3)))
   )
-  (gr_text J1 (at 152.7 43.3) (layer Eco1.User)
+  (gr_text J1 (at 152.7 42.7) (layer Eco1.User)
     (effects (font (size 1 1) (thickness 0.2)))
   )
@@
     (effects (font (size 1 1) (thickness 0.2)))
   )
-  (gr_text C2 (at 149.8 47.8) (layer Eco1.User)
+  (gr_text C2 (at 146.8 48.7) (layer Eco1.User)
     (effects (font (size 1 1) (thickness 0.2)))
   )
@@
   (gr_circle (center 147 22) (end 147 19.2) (layer Eco1.User) (width 0.15))
   (gr_circle (center 165 57) (end 165 54.2) (layer Eco1.User) (width 0.15))
-  (gr_line (start 153.4 44) (end 153.4 45.6) (layer Eco1.User) (width 0.15))
-  (gr_line (start 150.2 44) (end 153.4 44) (layer Eco1.User) (width 0.15))
-  (gr_line (start 150.2 45.6) (end 150.2 44) (layer Eco1.User) (width 0.15))
+  (gr_line (start 152.3 46) (end 152.3 47.6) (layer Eco1.User) (width 0.15))
+  (gr_line (start 149.1 46) (end 152.3 46) (layer Eco1.User) (width 0.15))
+  (gr_line (start 149.1 47.6) (end 149.1 46) (layer Eco1.User) (width 0.15))
   (gr_line (start 159.1 50.9) (end 159.7 50.9) (layer Eco1.User) (width 0.15))
   (gr_line (start 159.7 49.7) (end 159.1 49.7) (layer Eco1.User) (width 0.15))
