File: hardware/led_driver.sch (KiCad schematic (older format))
At the start: 43 parts, among them J1 CONN_01X01, J2 CONN_01X05, J3 CONN_01X05, J4 CONN_01X08, J5 CONN_01X08, J6 CONN_01X08, J7 CONN_01X08, J8 AVR-PDI-6A, P1 USB_A, U1 AP3211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

Commit message: Sorted out library references
Parts:
- removed J3: CONN_01X05, Primayer:B5B-ZR-SM4-TF, symbol CONN_01X05
- added J3: CONN_01X08, Kuro:B8B-ZR-SM4-TF, symbol CONN_01X08
- added U8: ASEK-32.768kHz, Kuro:Crystal-3.2x2.5-ASEK-Series-Abracon, symbol ASEK-32.768kHz
- J2: footprint Primayer:B5B-ZR-SM4-TF -> Kuro:B5B-ZR-SM4-TF
- J4, J5, J6, J7: footprint Primayer:B8B-ZR-SM4-TF -> Kuro:B8B-ZR-SM4-TF
- J8: footprint Primayer:3x2_1.27mm_SMD_header -> Kuro:3x2_1.27mm_SMD_header
- P1: footprint Primayer:Molex_47346-0001_Micro_USB_SMT -> Kuro:Molex_47346-0001_Micro_USB_SMT
- U7: footprint Primayer:KT3225T -> Kuro:KT3225T
Connections:
- net +3V3: now also J8.2, J3.7 (P7), U8.4 (Vdd)
- net +5V: now also J3.1 (P1)
- net EXP_ANA: now also J3.2 (P2)
- net GND: now also J8.6, J3.8 (P8), U8.2 (GND)
- net PDI_C: now also J8.5
- net PDI_D: now also J8.1
- net SCL: now also R5.2, U2.4 (SCLK), U4.15 (IN2/SCL/XCK0/OC4AHS/OC4B/PC1), J3.4 (P4); no longer J2.3 (P3), U4.11 (IN2/SCK/XCK0/OC5B/OC4CHS/OC4B/PC5), U5.14 (SCL), U6.14 (SCL)
- net at U4.19 (PR1/XTAL1/TOSC1/EXTCLK/AC0OUT), U7.5 (CLK): now also U8.3 (OUT)
- net EXP_RX_SDA renamed SDA
- net SDA: now also J3.3 (P3); no longer U4.14 (IN0/RXD0/~OC4BLS~/OC4C/PC2)
- removed net EXP_TX_SCL: R5.2, U2.4 (SCLK), U4.13 (IN3/TXD0/OC4BHS/OC4D/PC3), U4.15 (IN2/SCL/XCK0/OC4AHS/OC4B/PC1)
- new net RX: J3.6 (P6), U4.14 (IN0/RXD0/~OC4BLS~/OC4C/PC2)
- new net SCK: J2.3 (P3), U4.11 (IN2/SCK/XCK0/OC5B/OC4CHS/OC4B/PC5), U5.14 (SCL), U6.14 (SCL)
- new net TX: J3.5 (P5), U4.13 (IN3/TXD0/OC4BHS/OC4D/PC3)
- no-connect marks 19 -> 20
Other:
- moved on the sheet: C5, C6, J1, L2, R4, R5, U2
