File: hardware/led_driver.sch (KiCad schematic (older format))
At the start: 44 parts, among them J1 CONN_01X01, J2 CONN_01X05, J3 CONN_01X08, J4 CONN_01X08, J5 CONN_01X08, J6 CONN_01X08, J7 CONN_01X08, J8 AVR-PDI-6A, J9 USB_A, U1 AP3211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

Commit message: RDA read OK
Parts:
- J2: BOM_PartNo (none) -> B5B-ZR-SM4-TF
- J3, J4, J5, J6, J7: BOM_PartNo (none) -> B8B-ZR-SM4-TF
- J9: symbol USB_A -> USB_A-RESCUE-led_driver
Changed lines of the file:
@@
 $EndComp
 $Comp
-L USB_A J9
+L USB_A-RESCUE-led_driver J9
 U 1 1 57FF5D2F
 P 900 1400
@@
 F 2 "Kuro:B8B-ZR-SM4-TF" H 10400 2700 50  0001 C CNN
 F 3 "" H 10400 2700 50  0000 C CNN
+F 4 "B8B-ZR-SM4-TF" H 10400 2700 60  0001 C CNN "BOM_PartNo"
 	1    10400 2700
 	1    0    0    -1
@@
 F 2 "Kuro:B8B-ZR-SM4-TF" H 10900 3600 50  0001 C CNN
 F 3 "" H 10900 3600 50  0000 C CNN
+F 4 "B8B-ZR-SM4-TF" H 10900 3600 60  0001 C CNN "BOM_PartNo"
 	1    10900 3600
 	1    0    0    -1
@@
 F 2 "Kuro:B8B-ZR-SM4-TF" H 10400 4900 50  0001 C CNN
 F 3 "" H 10400 4900 50  0000 C CNN
+F 4 "B8B-ZR-SM4-TF" H 10400 4900 60  0001 C CNN "BOM_PartNo"
 	1    10400 4900
 	1    0    0    -1
@@
 F 2 "Kuro:B8B-ZR-SM4-TF" H 10900 5800 50  0001 C CNN
 F 3 "" H 10900 5800 50  0000 C CNN
+F 4 "B8B-ZR-SM4-TF" H 10900 5800 60  0001 C CNN "BOM_PartNo"
 	1    10900 5800
 	1    0    0    -1
@@
 F 2 "Kuro:B5B-ZR-SM4-TF" H 7550 4650 50  0001 C CNN
 F 3 "" H 7550 4650 50  0000 C CNN
+F 4 "B5B-ZR-SM4-TF" H 7550 4650 60  0001 C CNN "BOM_PartNo"
 	1    7550 4650
 	1    0    0    -1
@@
 F 2 "Kuro:B8B-ZR-SM4-TF" H 7550 5750 50  0001 C CNN
 F 3 "" H 7550 5750 50  0000 C CNN
+F 4 "B8B-ZR-SM4-TF" H 7550 5750 60  0001 C CNN "BOM_PartNo"
 	1    7550 5750
 	1    0    0    -1
